File: Board/Expand_v1_02.sch (EAGLE design)
At the start: 58 parts, among them U1 74LS541N, U10 7400N, U11 MC34063, U12 LM2596S, U2 74LS243N, U3 7407N, U4 74LS541N, U5 74LS541N, U7 74LS245N, U8 74AS573N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

Commit message: v1.0 Rev2 PCB Added
Added new board version, added notes, updated BOM.
Parts:
- removed X1: S4B-ZR, con-jst:S4B-ZR
- added J1: 22-05-7048-04, con-molex:22-05-7048-04
- added TP1, TP2, TP3, TP4: PTR1B2,54, testpad:PTR1B2,54
- C10, C11, C12, C17, C3, C4, C5, C6, C7, C8, C9: value (none) -> 100nF
- C13: value (none) -> 220uF
- R1, R15, R16, R2: value (none) -> 330R
- R10, R11, R3, R4, R5, R6, R7, R8, R9: value (none) -> 4.7k
- R12: device rcl:R-US_0207/7 -> rcl:R-US_0207/10
- R13: value 10k -> (none); device rcl:R-US_0207/7 -> pot:TRIM_US-RJ9W
- S1: value (none) -> 200MSP1T3B4M6RE
- U1, U4, U5: value 74LS541N -> 74F541N
- U10: value 7400N -> 74LS00N
- U2: value 74LS243N -> 74ALS243N
- U3: value 7407N -> 74LS07N
- U6: value (none) -> 22V10
- U7: value 74LS245N -> 74F245N
- U8: value 74AS573N -> 74LS573N
- U9: value 74S153N -> 74F153N
- renumbered U$1 to CONN2, U$2 to CONN3
Connections:
- net +12V: now also J1-4.S; no longer X1-4.1
- net -12V: now also TP1.TP
- net GND: now also J1-2.S, J1-3.S, R13.E, R13.S, TP2.TP, TP3.TP; no longer R13.1, X1-2.1, X1-3.1
- net N$22: now also R13.A; no longer R13.2
- net VCC: now also J1-1.S, TP4.TP; no longer X1-1.1
Other:
- moved on the sheet: R12
